Commit message: good urdf with tool

File: staubli_tx2_90_support/urdf/tx2_90l_macro.xacro (robot description, xacro)
@@ -106,4 +106,49 @@
         <geometry>
           <mesh filename="package://staubli_tx2_90_support/meshes/tx2_90/collision/link_6.stl"/>
+        </geometry>
+      </collision>
+    </link>
+    <link name="${prefix}link_tool">
+      <visual>
+        <origin xyz="0 0 0" rpy="0  0 0"/>
+        <geometry>
+          <mesh filename="package://staubli_tx2_90_support/meshes/tx2_90l/visual/tool_meter.stl"/>
+        </geometry>
+        <xacro:material_staubli_ral_grey_aluminium />
+      </visual>
+      <collision>
+        <origin xyz="0 0 0" rpy="${radians(90)} 0 0"/>
+        <geometry>
+          <mesh filename="package://staubli_tx2_90_support/meshes/tx2_90l/collision/convex/tool/one_tool_meter.obj"/>
+        </geometry>
+      </collision>
+    </link>
+    <link name="${prefix}link_finger1">
+      <visual>
+        <origin xyz="0 0 0" rpy="0 0 0"/>
+        <geometry>
+          <mesh filename="package://staubli_tx2_90_support/meshes/tx2_90l/visual/finger_meter.stl"/>
+        </geometry>
+        <xacro:material_staubli_ral_grey_aluminium />
+      </visual>
+      <collision>
+        <origin xyz="0 0 0" rpy="${radians(90)} 0 0"/>
+        <geometry>
+          <mesh filename="package://staubli_tx2_90_support/meshes/tx2_90l/collision/convex/finger/one_finger_meter.obj"/>
+        </geometry>
+      </collision>
+    </link>
+    <link name="${prefix}link_finger2">
+      <visual>
+        <origin xyz="0 0 0" rpy="0 0 ${pi}"/>
+        <geometry>
+          <mesh filename="package://staubli_tx2_90_support/meshes/tx2_90l/visual/finger_meter.stl"/>
+        </geometry>
+        <xacro:material_staubli_ral_grey_aluminium />
+      </visual>
+      <collision>
+        <origin xyz="0 0 0" rpy="${radians(90)} 0 ${pi}"/>
+        <geometry>
+          <mesh filename="package://staubli_tx2_90_support/meshes/tx2_90l/collision/convex/finger/one_finger_meter.obj"/>
         </geometry>
       </collision>
@@ -161,4 +206,24 @@
       <limit lower="${radians(-270)}" upper="${radians(270)}" effort="11.0" velocity="${radians(630)}" />
     </joint>
+    <joint name="${prefix}join_tool" type="fixed">
+      <origin xyz="0 0 0" rpy="${radians(90)} 0 ${radians(-45)}"/>
+      <parent link="${prefix}link_6"/>
+      <child link="${prefix}link_tool"/>
+    </joint>
+    <joint name="${prefix}finger_joint1" type="prismatic">
+      <parent link="${prefix}link_tool"/>
+      <child link="${prefix}link_finger1"/>
+      <origin xyz="-0.006 0.28964 0.00756" rpy="${radians(-70)} 0 0"/>
+      <axis xyz="1 0 0"/>
+      <limit effort="20" lower="0.0" upper="0.006" velocity="0.2"/>
+    </joint>
+    <joint name="${prefix}finger_joint2" type="prismatic">
+      <parent link="${prefix}link_tool"/>
+      <child link="${prefix}link_finger2"/>
+      <origin xyz="0.006 0.28964 0.00756" rpy="${radians(-70)} 0 0"/>
+      <axis xyz="-1 0 0"/>
+      <limit effort="20" lower="0.0" upper="0.006" velocity="0.2"/>
+      <mimic joint="${prefix}finger_joint1" />
+    </joint>
     <!-- ROS-Industrial 'base' frame: base_link to Staubli World Coordinates transform -->
     <link name="${prefix}base" />

Commit message: changes cao

File: staubli_tx2_90_support/urdf/tx2_90l_macro.xacro (robot description, xacro)
@@ -111,14 +111,14 @@
     <link name="${prefix}link_tool">
       <visual>
-        <origin xyz="0 0 0" rpy="0  0 0"/>
-        <geometry>
-          <mesh filename="package://staubli_tx2_90_support/meshes/tx2_90l/visual/tool_meter.stl"/>
-        </geometry>
-        <xacro:material_staubli_ral_grey_aluminium />
-      </visual>
-      <collision>
-        <origin xyz="0 0 0" rpy="${radians(90)} 0 0"/>
-        <geometry>
-          <mesh filename="package://staubli_tx2_90_support/meshes/tx2_90l/collision/convex/tool/one_tool_meter.obj"/>
+        <origin xyz="0 0 0" rpy="${radians(-90)} 0 0"/>
+        <geometry>
+          <mesh filename="package://staubli_tx2_90_support/meshes/tx2_90l/visual/true_tool_meter.stl"/>
+        </geometry>
+        <xacro:material_staubli_ral_grey_aluminium />
+      </visual>
+      <collision>
+        <origin xyz="0 0 0" rpy="0 0 0"/>
+        <geometry>
+          <mesh filename="package://staubli_tx2_90_support/meshes/tx2_90l/collision/convex/tool/true_tool_meter.obj"/>
         </geometry>
       </collision>
@@ -164,5 +164,5 @@
       (2) effort limit = 75 Nm if wall mounted -->
       <!-- nominal velocity limits are used -->
-      <limit lower="${radians(-180)}" upper="${radians(180)}" effort="318.0" velocity="${radians(225)}" />
+      <limit lower="${-3.0}" upper="${0.0}" effort="318.0" velocity="${radians(225)}" />
     </joint>
     <joint name="${prefix}joint_2" type="revolute">
@@ -172,5 +172,5 @@
       <axis xyz="0 1 0"/>
       <!-- nominal velocity limits are used -->
-      <limit lower="${radians(-130)}" upper="${radians(147.5)}" effort="130.0" velocity="${radians(180)}" />
+      <limit lower="${-0.7}" upper="${1.57}" effort="130.0" velocity="${radians(180)}" />
     </joint>
     <joint name="${prefix}joint_3" type="revolute">
@@ -180,5 +180,5 @@
       <axis xyz="0 1 0"/>
       <!-- nominal velocity limits are used -->
-      <limit lower="${radians(-145)}" upper="${radians(145)}" effort="65.0" velocity="${radians(270)}" />
+      <limit lower="${-0.7}" upper="${2.53}" effort="65.0" velocity="${radians(270)}" />
     </joint>
     <joint name="${prefix}joint_4" type="revolute">
@@ -188,5 +188,5 @@
       <axis xyz="0 0 1"/>
       <!-- nominal velocity limits are used -->
-      <limit lower="${radians(-270)}" upper="${radians(270)}" effort="34.0" velocity="${radians(450)}" />
+      <limit lower="${-2.27}" upper="${2.27}" effort="34.0" velocity="${radians(450)}" />
     </joint>
     <joint name="${prefix}joint_5" type="revolute">
@@ -196,5 +196,5 @@
       <axis xyz="0 1 0"/>
       <!-- nominal velocity limits are used -->
-      <limit lower="${radians(-115)}" upper="${radians(140)}" effort="29.0" velocity="${radians(370)}" />
+      <limit lower="${-2}" upper="${2.39}" effort="29.0" velocity="${radians(370)}" />
     </joint>
     <joint name="${prefix}joint_6" type="revolute">
@@ -204,7 +204,7 @@
       <axis xyz="0 0 1"/>
       <!-- nominal velocity limits are used -->
-      <limit lower="${radians(-270)}" upper="${radians(270)}" effort="11.0" velocity="${radians(630)}" />
-    </joint>
-    <joint name="${prefix}join_tool" type="fixed">
+      <limit lower="${radians(-180)}" upper="${radians(180)}" effort="11.0" velocity="${radians(630)}" />
+    </joint>
+    <joint name="${prefix}joint_tool" type="fixed">
       <origin xyz="0 0 0" rpy="${radians(90)} 0 ${radians(-45)}"/>
       <parent link="${prefix}link_6"/>
@@ -214,5 +214,5 @@
       <parent link="${prefix}link_tool"/>
       <child link="${prefix}link_finger1"/>
-      <origin xyz="-0.006 0.28964 0.00756" rpy="${radians(-70)} 0 0"/>
+      <origin xyz="-0.006 0.28498 0.00783" rpy="${radians(-70)} 0 0"/>
       <axis xyz="1 0 0"/>
       <limit effort="20" lower="0.0" upper="0.006" velocity="0.2"/>
@@ -221,5 +221,5 @@
       <parent link="${prefix}link_tool"/>
       <child link="${prefix}link_finger2"/>
-      <origin xyz="0.006 0.28964 0.00756" rpy="${radians(-70)} 0 0"/>
+      <origin xyz="0.006 0.28498 0.00783" rpy="${radians(-70)} 0 0"/>
       <axis xyz="-1 0 0"/>
       <limit effort="20" lower="0.0" upper="0.006" velocity="0.2"/>
